Commit message: WIP Fixed URDF Scara robot

File: data/scara_robot.urdf (robot description, URDF)
Before this commit: robot scara_robot, 6 links, 5 joints
Links:
- removed link end_effector
- removed link link3
- removed link link4
- added link link_end_effector; visual cylinder length=0.2 radius=0.02
- link base_link: mass 1.0 -> None; geometry visual box size=0.12 0.12 0.12
- link link1: mass 0.5 -> None; geometry visual box size=0.350 0.09 0.025
- link link2: mass 0.3 -> None; geometry visual box size=0.450 0.09 0.025
Joints:
- removed joint joint3
- removed joint joint4
- removed joint joint5
- added joint end_effector: type prismatic, parent link2, child link_end_effector, origin xyz=0.45 0 0 rpy=0 0 0, axis 0 0 -1, limit lower=-0.16 upper=0.038 effort=5 velocity=0.2
- joint joint1: origin xyz=0 0 0.05 rpy=0 0 0 -> xyz=0 0 0.06 rpy=0 0 0
- joint joint2: origin xyz=0.3 0 0 rpy=0 0 0 -> xyz=0.35 0 0 rpy=0 0 0

Commit message: Fix URDFs

File: data/scara_robot.urdf (robot description, URDF)
Before this commit: robot scara_robot, 4 links, 3 joints
Joints:
- joint end_effector: limit lower=-0.16 upper=0.038 effort=5 velocity=0.2 -> lower=0.038 upper=0.16 effort=5 velocity=0.2

File: data/simple_diff_drive_robot.urdf (robot description, URDF)
Before this commit: robot simple_diff_drive_robot, 4 links, 3 joints
Links:
- link left_wheel: geometry visual cylinder length=0.05 radius=0.1
- link right_wheel: geometry visual cylinder length=0.05 radius=0.10
Joints:
- joint caster_joint: origin xyz=0.15 0 0.01 rpy=0 0 0 -> xyz=0.15 0 -0.05 rpy=0 0 0
- joint left_wheel_joint: origin xyz=-0.15 0.15 0.025 rpy=0 1.5708 0 -> xyz=-0.15 0.15 0.025 rpy=1.5708 0 0
- joint right_wheel_joint: origin xyz=-0.15 -0.15 0.025 rpy=0 1.5708 0 -> xyz=-0.15 -0.15 0.025 rpy=1.5708 0 0

File: data/simple_revolute_robot.urdf (robot description, URDF)
Before this commit: robot simple_revolute_robot, 3 links, 2 joints
Links:
- removed link end_effector_link
Joints:
- removed joint end_effector_joint
