Commit message: WIP

File: data/cartesian_robot.urdf (robot description, URDF)
Before this commit: robot cartesian_robot_full, 5 links, 4 joints
Links:
- removed link base_link
- removed link end_effector_link
- removed link link1
- removed link link2
- removed link link3
- added link frame2; visual box size=1.1 0.1 0.1
- added link link_x; visual box size=0.1 1.0 0.1
- added link link_y; visual box size=0.15 0.15 0.15
- added link link_z; visual cylinder length=0.3 radius=0.04
Joints:
- removed joint end_effector
- removed joint joint1
- removed joint joint2
- removed joint joint3
- added joint joint_x: type prismatic, parent frame2, child link_x, origin xyz=0 0 0 rpy=0 0 0, axis 1 0 0, limit lower=-0.5 upper=0.5 effort=100 velocity=10
- added joint joint_y: type prismatic, parent link_x, child link_y, origin xyz=0 0 0 rpy=0 0 0, axis 0 1 0, limit lower=-0.45 upper=0.45 effort=100 velocity=10
- added joint joint_z: type prismatic, parent link_y, child link_z, origin xyz=0 0 0 rpy=0 0 0, axis 0 0 1, limit lower=-0.1 upper=0.0 effort=100 velocity=10
