Commit message: Mesh, STL, applications
- Add Mesh file shared both by MeshManager and GeometryRender
- Add path prefix for loading STL files and namespacing the dictionnary
- Rename demos folder to applications

File: data/T12.urdf (robot description, URDF)
Before this commit: robot T12, 37 links, 36 joints
Links:
- link Ankle1: geometry collision mesh filename=Ankle1.STL; visual mesh filename=Ankle1.STL
- link Ankle2: geometry collision mesh filename=Ankle2.STL; visual mesh filename=Ankle2.STL
- link Ankle3: geometry collision mesh filename=Ankle3.STL; visual mesh filename=Ankle3.STL
- link Ankle4: geometry collision mesh filename=Ankle4.STL; visual mesh filename=Ankle4.STL
- link Ankle5: geometry collision mesh filename=Ankle5.STL; visual mesh filename=Ankle5.STL
- link Ankle6: geometry collision mesh filename=Ankle6.STL; visual mesh filename=Ankle6.STL
- link Body: geometry collision mesh filename=Body.STL; visual mesh filename=Body.STL
- link Foot1: geometry collision mesh filename=Foot1.STL; visual mesh filename=Foot1.STL
- link Foot2: geometry collision mesh filename=Foot2.STL; visual mesh filename=Foot2.STL
- link Foot3: geometry collision mesh filename=Foot3.STL; visual mesh filename=Foot3.STL
- link Foot4: geometry collision mesh filename=Foot4.STL; visual mesh filename=Foot4.STL
- link Foot5: geometry collision mesh filename=Foot5.STL; visual mesh filename=Foot5.STL
- link Foot6: geometry collision mesh filename=Foot6.STL; visual mesh filename=Foot6.STL
- link Hip1: geometry collision mesh filename=Hip1.STL; visual mesh filename=Hip1.STL
- link Hip2: geometry collision mesh filename=Hip2.STL; visual mesh filename=Hip2.STL
- link Hip3: geometry collision mesh filename=Hip3.STL; visual mesh filename=Hip3.STL
- link Hip4: geometry collision mesh filename=Hip4.STL; visual mesh filename=Hip4.STL
- link Hip5: geometry collision mesh filename=Hip5.STL; visual mesh filename=Hip5.STL
- link Hip6: geometry collision mesh filename=Hip6.STL; visual mesh filename=Hip6.STL
- link Knee1: geometry collision mesh filename=Knee1.STL; visual mesh filename=Knee1.STL
- link Knee2: geometry collision mesh filename=Knee2.STL; visual mesh filename=Knee2.STL
- link Knee3: geometry collision mesh filename=Knee3.STL; visual mesh filename=Knee3.STL
- link Knee4: geometry collision mesh filename=Knee4.STL; visual mesh filename=Knee4.STL
- link Knee5: geometry collision mesh filename=Knee5.STL; visual mesh filename=Knee5.STL
- link Knee6: geometry collision mesh filename=Knee6.STL; visual mesh filename=Knee6.STL
- link Shin1: geometry collision mesh filename=Shin1.STL; visual mesh filename=Shin1.STL
- link Shin2: geometry collision mesh filename=Shin2.STL; visual mesh filename=Shin2.STL
- link Shin3: geometry collision mesh filename=Shin3.STL; visual mesh filename=Shin3.STL
- link Shin4: geometry collision mesh filename=Shin4.STL; visual mesh filename=Shin4.STL
- link Shin5: geometry collision mesh filename=Shin5.STL; visual mesh filename=Shin5.STL
- link Shin6: geometry collision mesh filename=Shin6.STL; visual mesh filename=Shin6.STL
- link Thigh1: geometry collision mesh filename=Thigh1.STL; visual mesh filename=Thigh1.STL
- link Thigh2: geometry collision mesh filename=Thigh2.STL; visual mesh filename=Thigh2.STL
- link Thigh3: geometry collision mesh filename=Thigh3.STL; visual mesh filename=Thigh3.STL
- link Thigh4: geometry collision mesh filename=Thigh4.STL; visual mesh filename=Thigh4.STL
- link Thigh5: geometry collision mesh filename=Thigh5.STL; visual mesh filename=Thigh5.STL
- link Thigh6: geometry collision mesh filename=Thigh6.STL; visual mesh filename=Thigh6.STL

Commit message: WIP

File: data/T12.urdf (robot description, URDF)
Before this commit: robot T12, 37 links, 36 joints
Links:
- link Ankle1: geometry collision mesh filename=T12/Ankle1.STL; visual mesh filename=T12/Ankle1.STL
- link Ankle2: geometry collision mesh filename=T12/Ankle2.STL; visual mesh filename=T12/Ankle2.STL
- link Ankle3: geometry collision mesh filename=T12/Ankle3.STL; visual mesh filename=T12/Ankle3.STL
- link Ankle4: geometry collision mesh filename=T12/Ankle4.STL; visual mesh filename=T12/Ankle4.STL
- link Ankle5: geometry collision mesh filename=T12/Ankle5.STL; visual mesh filename=T12/Ankle5.STL
- link Ankle6: geometry collision mesh filename=T12/Ankle6.STL; visual mesh filename=T12/Ankle6.STL
- link Body: geometry collision mesh filename=T12/Body.STL; visual mesh filename=T12/Body.STL
- link Foot1: geometry collision mesh filename=T12/Foot1.STL; visual mesh filename=T12/Foot1.STL
- link Foot2: geometry collision mesh filename=T12/Foot2.STL; visual mesh filename=T12/Foot2.STL
- link Foot3: geometry collision mesh filename=T12/Foot3.STL; visual mesh filename=T12/Foot3.STL
- link Foot4: geometry collision mesh filename=T12/Foot4.STL; visual mesh filename=T12/Foot4.STL
- link Foot5: geometry collision mesh filename=T12/Foot5.STL; visual mesh filename=T12/Foot5.STL
- link Foot6: geometry collision mesh filename=T12/Foot6.STL; visual mesh filename=T12/Foot6.STL
- link Hip1: geometry collision mesh filename=T12/Hip1.STL; visual mesh filename=T12/Hip1.STL
- link Hip2: geometry collision mesh filename=T12/Hip2.STL; visual mesh filename=T12/Hip2.STL
- link Hip3: geometry collision mesh filename=T12/Hip3.STL; visual mesh filename=T12/Hip3.STL
- link Hip4: geometry collision mesh filename=T12/Hip4.STL; visual mesh filename=T12/Hip4.STL
- link Hip5: geometry collision mesh filename=T12/Hip5.STL; visual mesh filename=T12/Hip5.STL
- link Hip6: geometry collision mesh filename=T12/Hip6.STL; visual mesh filename=T12/Hip6.STL
- link Knee1: geometry collision mesh filename=T12/Knee1.STL; visual mesh filename=T12/Knee1.STL
- link Knee2: geometry collision mesh filename=T12/Knee2.STL; visual mesh filename=T12/Knee2.STL
- link Knee3: geometry collision mesh filename=T12/Knee3.STL; visual mesh filename=T12/Knee3.STL
- link Knee4: geometry collision mesh filename=T12/Knee4.STL; visual mesh filename=T12/Knee4.STL
- link Knee5: geometry collision mesh filename=T12/Knee5.STL; visual mesh filename=T12/Knee5.STL
- link Knee6: geometry collision mesh filename=T12/Knee6.STL; visual mesh filename=T12/Knee6.STL
- link Shin1: geometry collision mesh filename=T12/Shin1.STL; visual mesh filename=T12/Shin1.STL
- link Shin2: geometry collision mesh filename=T12/Shin2.STL; visual mesh filename=T12/Shin2.STL
- link Shin3: geometry collision mesh filename=T12/Shin3.STL; visual mesh filename=T12/Shin3.STL
- link Shin4: geometry collision mesh filename=T12/Shin4.STL; visual mesh filename=T12/Shin4.STL
- link Shin5: geometry collision mesh filename=T12/Shin5.STL; visual mesh filename=T12/Shin5.STL
- link Shin6: geometry collision mesh filename=T12/Shin6.STL; visual mesh filename=T12/Shin6.STL
- link Thigh1: geometry collision mesh filename=T12/Thigh1.STL; visual mesh filename=T12/Thigh1.STL
- link Thigh2: geometry collision mesh filename=T12/Thigh2.STL; visual mesh filename=T12/Thigh2.STL
- link Thigh3: geometry collision mesh filename=T12/Thigh3.STL; visual mesh filename=T12/Thigh3.STL
- link Thigh4: geometry collision mesh filename=T12/Thigh4.STL; visual mesh filename=T12/Thigh4.STL
- link Thigh5: geometry collision mesh filename=T12/Thigh5.STL; visual mesh filename=T12/Thigh5.STL
- link Thigh6: geometry collision mesh filename=T12/Thigh6.STL; visual mesh filename=T12/Thigh6.STL
