Commit message: Add generated URDF files

File: data/robot_6axis.urdf (robot description, URDF)
Before this commit: robot robot_6axes, 7 links, 6 joints
Links:
- added link flange
- added link tool0
- link base_link: geometry collision cylinder length=0.1 radius=0.15; visual cylinder length=0.006 radius=0.008
- link link1: geometry collision cylinder length=0.3 radius=0.08; visual cylinder length=0.01 radius=0.0765
- link link2: geometry collision cylinder length=0.35 radius=0.06; visual cylinder length=0.008 radius=0.0565
- link link3: geometry collision cylinder length=0.3 radius=0.05; visual cylinder length=0.006 radius=0.0455
- link link4: geometry collision cylinder length=0.08 radius=0.04; visual cylinder length=0.045 radius=0.04
- link link5: geometry collision cylinder length=0.08 radius=0.035; visual cylinder length=0.005 radius=0.0335
- link link6: mass 0.5 -> 0.4; geometry collision cylinder length=0.044 radius=0.032; visual box size=0.024 0.03 0.02
Joints:
- added joint flange_to_tool0: type fixed, parent flange, child tool0, origin xyz=0 0 0 rpy=0 0 0
- added joint link6_to_flange: type fixed, parent link6, child flange, origin xyz=0 0 0.044 rpy=0 0 0
