Commit message: Add generated URDF files

File: data/robot_6axis_vacuum.urdf (robot description, URDF)
Before this commit: robot robot_6axes, 9 links, 8 joints
Links:
- removed link flange
- removed link tool0
- link link6: mass 0.4 -> 0.5; geometry collision box size=0.06 0.03 0.03; visual box size=0.024 0.03 0.02
Joints:
- removed joint flange_to_tool0
- removed joint link6_to_flange
